File: opentx.brd (EAGLE design)
At the start: 169 x 41 mm, 9 parts, among them IC1 STM32F205VET

Commit message: pcb
Parts:
- added PAD1, PAD10, PAD11, PAD12, PAD13, PAD14, PAD15, PAD16, PAD17, PAD18, PAD19, PAD2, PAD20, PAD21, PAD22, PAD23, PAD3, PAD4, PAD5, PAD6, PAD7, PAD8, PAD9: (no value), wirepad:SMD1,27-2,54
- added U1: 24LC256, SparkFun-IC-Memory:SO08
Connections:
- new net N$1: U1.1, U1.8
- new net N$10: PAD16.1
- new net N$2: U1.2, U1.3, U1.4
- new net N$7: PAD7.1
- new net N$8: PAD8.1
- new net N$9: PAD15.1
- net ADC_STICK_LH: now also PAD5.1
- net ADC_STICK_LV: now also PAD6.1
- net ADC_STICK_RH: now also PAD13.1
- net ADC_STICK_RV: now also PAD14.1
- net BACKLIGHT: now also PAD21.1
- net I2C_SDA: now also U1.5, U1.6
- net I2C_WP: now also U1.7
- net LCD_A0: now also PAD18.1
- net LCD_CLK: now also PAD19.1
- net LCD_MOSI: now also PAD17.1
- net LCD_RST: now also PAD20.1
- net TRIMS_LHL: now also PAD4.1
- net TRIMS_LHR: now also PAD3.1
- net TRIMS_LVD: now also PAD1.1
- net TRIMS_LVU: now also PAD2.1
- net TRIMS_RHL: now also PAD12.1
- net TRIMS_RHR: now also PAD11.1
- net TRIMS_RVD: now also PAD9.1
- net TRIMS_RVU: now also PAD10.1

Commit message: pcb
Parts:
- added PAD24, PAD25, PAD26, PAD27, PAD28, PAD29, PAD30, PAD31, PAD32, PAD33: (no value), wirepad:SMD1,27-2,54
- added U$2: MICROSD_SPI_MODE, con-molex-microsd:MICRO_SD_CONNECTOR
- moved IC1 5.42 mm to (116.6, 12.5), turned to 180 degrees
Connections:
- net SD_CS: now also U$2.2
- net SD_MISO: now also U$2.7
- net SD_MOSI: now also U$2.3
- net SD_PRESENT: now also U$2.9
- net SD_SCK: now also U$2.5
- net SWITCHES_A_H: now also PAD26.1
- net SWITCHES_A_L: now also PAD24.1
- net SWITCHES_B_H: now also PAD25.1
- net SWITCHES_B_L: now also PAD27.1
- net SWITCHES_C_H: now also PAD29.1
- net SWITCHES_C_L: now also PAD28.1
- net SWITCHES_D_H: now also PAD31.1
- net SWITCHES_D_L: now also PAD30.1
- net SWITCHES_F: now also PAD32.1
- net SWITCHES_H: now also PAD33.1

Commit message: pcb
Parts:
- added J1: (no value), SparkFun-Connectors:USB-AB-MICRO-SMD
- added Y1: 32.768kHz, SparkFun-Clocks:CRYSTAL-SMD-2X6-CYL
- moved PAD33 42.3 mm to (63.0, 37.0)
- moved PAD32 41.7 mm to (65.5, 37.0)
- moved PAD31 41.0 mm to (68.0, 37.0)
- moved PAD30 40.4 mm to (70.5, 37.0)
- moved PAD29 39.8 mm to (73.0, 37.0)
- moved PAD28 39.2 mm to (75.5, 37.0)
- moved PAD27 38.6 mm to (78.0, 37.0)
- moved PAD26 38.1 mm to (80.5, 37.0)
- moved PAD25 37.5 mm to (83.0, 37.0)
- moved PAD24 37.0 mm to (85.5, 37.0)
- moved PAD23 13.4 mm to (96.5, 37.0)
- moved PAD22 12.5 mm to (99.0, 37.0)
- moved PAD21 11.6 mm to (101.5, 37.0)
- moved PAD20 10.7 mm to (104.0, 37.0)
- moved PAD19 9.80 mm to (106.5, 37.0)
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Connections:
- removed net N$10: PAD16.1
- removed net N$7: PAD7.1
- removed net N$8: PAD8.1
- removed net N$9: PAD15.1
- new net +3V3: PAD15.1, PAD7.1, U$2.4, U1.1, U1.8
- new net GND: J1.GND1, J1.SHLD1, J1.SHLD2, J1.SHLD3, PAD16.1, PAD8.1, U$2.6, U1.2, U1.3, U1.4
- net I2C_SCL: now also U1.6
- net I2C_SDA: no longer U1.6
- net N$1: now also IC1.8, Y1.X1; no longer U1.1, U1.8
- net N$2: now also IC1.9, Y1.X2; no longer U1.2, U1.3, U1.4
- net USB_DM: now also J1.D-1
- net USB_DP: now also J1.D+1
- net USB_VBUS: now also J1.VBUS1
Routing:
- net TRIMS_RHL: track 0.00 -> 103.2 mm
- net TRIMS_RHR: track 0.00 -> 100.2 mm
- net ADC_STICK_RV: track 0.00 -> 97.8 mm
- net ADC_STICK_RH: track 0.00 -> 94.8 mm
- net TRIMS_RVU: track 0.00 -> 90.8 mm
- net TRIMS_RVD: track 0.00 -> 87.8 mm
- net TRIMS_LHL: track 0.00 -> 51.2 mm, vias 0 -> 2
- net USB_VBUS: track 0.00 -> 43.8 mm
- net TRIMS_LVU: track 0.00 -> 43.8 mm
- net USB_DM: track 0.00 -> 42.2 mm
- net USB_DP: track 0.00 -> 41.0 mm
- net TRIMS_LVD: track 0.00 -> 40.8 mm
- net SD_MOSI: track 0.00 -> 33.8 mm
- net TRIMS_LHR: track 0.00 -> 32.8 mm
- net SD_CS: track 0.00 -> 26.0 mm
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
Commit message: pcb
Parts:
- added PAD34, PAD35: (no value), wirepad:SMD1,27-2,54
- added Y2: (no value), SparkFun-Clocks:HC49UP
- moved PAD4 10.0 mm to (151.0, 36.5)
- moved PAD2 5.00 mm to (143.5, 36.5)
- moved PAD3 5.00 mm to (148.5, 36.5)
- moved Y1 2.69 mm to (139.0, 15.5)
Connections:
- new net N$3: IC1.12, Y2.2
- new net N$4: IC1.13, Y2.1
Routing:
- net SWITCHES_A_H: track 0.00 -> 69.2 mm, vias 0 -> 2
- net SWITCHES_B_H: track 0.00 -> 49.2 mm
- net SWITCHES_B_L: track 0.00 -> 46.2 mm
- net SWITCHES_A_L: track 0.00 -> 42.8 mm
- net N$3: track 0.00 -> 18.1 mm
- net TRIMS_LHL: track 51.2 -> 61.2 mm
- net N$4: track 0.00 -> 7.92 mm
- net ADC_STICK_RV: track 97.8 -> 105.2 mm, vias 0 -> 2
- net TRIMS_LVD: track 40.8 -> 46.8 mm, vias 0 -> 2
- net ADC_STICK_RH: track 94.8 -> 100.2 mm, vias 0 -> 2
- net TRIMS_LHR: track 32.8 -> 37.8 mm
- net N$2: track 17.0 -> 13.5 mm
- net TRIMS_LVU: track 43.8 -> 45.8 mm, vias 0 -> 2
- net N$1: track 15.5 -> 17.0 mm

Commit message: scheme & photo
Parts:
- added PAD36, PAD37, PAD38, PAD39, PAD40, PAD41, PAD42, PAD43, PAD44, PAD45, PAD46, PAD47, PAD48: (no value), wirepad:SMD1,27-2,54
Connections:
- net ADC_STICK_LH renamed ADC_STICK_LH_PA3
- net ADC_STICK_LV renamed ADC_STICK_LV_PA2
- net ADC_STICK_RH renamed ADC_STICK_RH_PA1
- net ADC_STICK_RV renamed ADC_STICK_RV_PA0
- net BACKLIGHT renamed BACKLIGHT_PD13
- net LCD_A0 renamed LCD_A0_PC11
- net LCD_CLK renamed LCD_CLK_PC10
- net LCD_MOSI renamed LCD_MOSI_PC12
- net LCD_RST renamed LCD_RST_PD12
- net SD_CS renamed SD_CS_PB12
- net SD_MISO renamed SD_MISO_PB14
- net SD_MOSI renamed SD_MOSI_PB15
- net SD_PRESENT renamed SD_PRESENT_PD9
- net SD_SCK renamed SD_SCK_PB13
- net TRIMS_LHL renamed TRIMS_LHL_PD15
- net TRIMS_LHR renamed TRIMS_LHR_PC1
- net TRIMS_LVD renamed TRIMS_LVD_PE6
- net TRIMS_LVU renamed TRIMS_LVU_PE5
- net TRIMS_RHL renamed TRIMS_RHL_PE3
- net TRIMS_RHR renamed TRIMS_RHR_PE4
- net TRIMS_RVD renamed TRIMS_RVD_PC3
- net TRIMS_RVU renamed TRIMS_RVU_PC2
- net USB_DM renamed USB_DM_PA11
- net USB_DP renamed USB_DP_PA12
- net USB_VBUS renamed USB_VBUS_PA9
- removed net ADC_POT1: IC1.31
- removed net ADC_POT2: IC1.35
- removed net ENC_A: IC1.40
- removed net ENC_B: IC1.42
- removed net EXTMODULE_PWR: IC1.55
- removed net EXTMODULE_TX: IC1.32
- removed net INTMODULE_PWR: IC1.63
- removed net INTMODULE_TX: IC1.69
- removed net KEYS_ENTER: IC1.41
- removed net KEYS_EXIT: IC1.83
- removed net KEYS_MENU: IC1.88
- removed net KEYS_PAGE: IC1.84
- removed net LCD_NCS: IC1.77
- new net ADC_POT1_PA6: IC1.31, PAD47.1
- new net ADC_POT2_PB0: IC1.35, PAD48.1
- new net ENC_A_PE9: IC1.40, PAD40.1
- new net ENC_B_PE11: IC1.42, PAD41.1
- new net EXTMODULE_PWR_PD8: IC1.55, PAD45.1
- new net EXTMODULE_TX_PA7: IC1.32, PAD44.1
- new net INTMODULE_PWR_PC6: IC1.63, PAD42.1
- new net INTMODULE_TX_PA10: IC1.69, PAD43.1
- new net KEYS_ENTER_PE10: IC1.41, PAD39.1
- new net KEYS_EXIT_PD2: IC1.83, PAD38.1
- new net KEYS_MENU_PD7: IC1.88, PAD36.1
- new net KEYS_PAGE_PD3: IC1.84, PAD37.1
- new net LCD_NCS_PA15: IC1.77, PAD22.1
- new net N$7: PAD46.1
- net SWITCHES_A_H: now also IC1.44; no longer IC1.91
Routing:
- net SWITCHES_A_H: track 69.2 -> 67.5 mm
