File: opentx.sch (EAGLE design)
At the start: 9 parts, among them IC1 STM32F205VET

Commit message: pcb
Parts:
- added PAD1, PAD10, PAD11, PAD12, PAD13, PAD14, PAD15, PAD16, PAD17, PAD18, PAD19, PAD2, PAD20, PAD21, PAD22, PAD23, PAD3, PAD4, PAD5, PAD6, PAD7, PAD8, PAD9: (no value), wirepad:SMD2
- added U1: 24LC256, SparkFun-IC-Memory:EEPROM-I2CSMD
Connections:
- new net N$1: U1.A0, U1.VCC
- new net N$10: PAD16.P
- new net N$2: U1.A1, U1.A2, U1.VSS
- new net N$7: PAD7.P
- new net N$8: PAD8.P
- new net N$9: PAD15.P
- net ADC_STICK_LH: now also PAD5.P
- net ADC_STICK_LV: now also PAD6.P
- net ADC_STICK_RH: now also PAD13.P
- net ADC_STICK_RV: now also PAD14.P
- net BACKLIGHT: now also PAD21.P
- net I2C_SDA: now also U1.SCL, U1.SDA
- net I2C_WP: now also U1.WP
- net LCD_A0: now also PAD18.P
- net LCD_CLK: now also PAD19.P
- net LCD_MOSI: now also PAD17.P
- net LCD_RST: now also PAD20.P
- net TRIMS_LHL: now also PAD4.P
- net TRIMS_LHR: now also PAD3.P
- net TRIMS_LVD: now also PAD1.P
- net TRIMS_LVU: now also PAD2.P
- net TRIMS_RHL: now also PAD12.P
- net TRIMS_RHR: now also PAD11.P
- net TRIMS_RVD: now also PAD9.P
- net TRIMS_RVU: now also PAD10.P

Commit message: pcb
Parts:
- added PAD24, PAD25, PAD26, PAD27, PAD28, PAD29, PAD30, PAD31, PAD32, PAD33: (no value), wirepad:SMD2
- added U$2: MICROSD_SPI_MODE, con-molex-microsd:MICROSD_SPI_MODE
Connections:
- net SD_CS: now also U$2./CS
- net SD_MISO: now also U$2.DO
- net SD_MOSI: now also U$2.DI
- net SD_PRESENT: now also U$2.CD(1)
- net SD_SCK: now also U$2.CLK
- net SWITCHES_A_H: now also PAD26.P
- net SWITCHES_A_L: now also PAD24.P
- net SWITCHES_B_H: now also PAD25.P
- net SWITCHES_B_L: now also PAD27.P
- net SWITCHES_C_H: now also PAD29.P
- net SWITCHES_C_L: now also PAD28.P
- net SWITCHES_D_H: now also PAD31.P
- net SWITCHES_D_L: now also PAD30.P
- net SWITCHES_F: now also PAD32.P
- net SWITCHES_H: now also PAD33.P

Commit message: pcb
Parts:
- added J1: (no value), SparkFun-Connectors:USB_AB_SMT
- added Y1: 32.768kHz, SparkFun-Clocks:CRYSTAL-32.768KHZSMD-2X6
Connections:
- removed net N$10: PAD16.P
- removed net N$7: PAD7.P
- removed net N$8: PAD8.P
- removed net N$9: PAD15.P
- new net +3V3: PAD15.P, PAD7.P, U$2.VDD, U1.A0, U1.VCC
- new net GND: J1.GND, J1.SHIELD, PAD16.P, PAD8.P, U$2.VSS, U1.A1, U1.A2, U1.VSS
- net I2C_SCL: now also U1.SCL
- net I2C_SDA: no longer U1.SCL
- net N$1: now also IC1MCU.PC14, Y1.1; no longer U1.A0, U1.VCC
- net N$2: now also IC1MCU.PC15, Y1.2; no longer U1.A1, U1.A2, U1.VSS
- net USB_DM: now also J1.D-
- net USB_DP: now also J1.D+
- net USB_VBUS: now also J1.VBUS
Other:
- moved on the sheet: PAD1, PAD2, PAD3, PAD4, PAD5, PAD6, PAD7, PAD8

Commit message: pcb
Parts:
- added PAD34, PAD35: (no value), wirepad:SMD2
- added Y2: (no value), SparkFun-Clocks:CRYSTALSMD-HC49UP
- PAD13: SPICEPREFIX (none) -> X
Connections:
- new net N$3: IC1MCU.OSC_IN, Y2.2
- new net N$4: IC1MCU.OSC_OUT, Y2.1
Other:
- moved on the sheet: PAD10, PAD11, PAD12, PAD13, PAD14, PAD2, PAD3, PAD4, PAD9

Commit message: scheme
Parts:
- added PAD36, PAD37, PAD38, PAD39, PAD40, PAD41, PAD42, PAD43, PAD44, PAD45, PAD46, PAD47, PAD48: (no value), wirepad:SMD2
Connections:
- net ADC_STICK_LH renamed ADC_STICK_LH_PA3
- net ADC_STICK_LV renamed ADC_STICK_LV_PA2
- net ADC_STICK_RH renamed ADC_STICK_RH_PA1
- net ADC_STICK_RV renamed ADC_STICK_RV_PA0
- net BACKLIGHT renamed BACKLIGHT_PD13
- net LCD_A0 renamed LCD_A0_PC11
- net LCD_CLK renamed LCD_CLK_PC10
- net LCD_MOSI renamed LCD_MOSI_PC12
- net LCD_RST renamed LCD_RST_PD12
- net SD_CS renamed SD_CS_PB12
- net SD_MISO renamed SD_MISO_PB14
- net SD_MOSI renamed SD_MOSI_PB15
- net SD_PRESENT renamed SD_PRESENT_PD9
- net SD_SCK renamed SD_SCK_PB13
- net TRIMS_LHL renamed TRIMS_LHL_PD15
- net TRIMS_LHR renamed TRIMS_LHR_PC1
- net TRIMS_LVD renamed TRIMS_LVD_PE6
- net TRIMS_LVU renamed TRIMS_LVU_PE5
- net TRIMS_RHL renamed TRIMS_RHL_PE3
- net TRIMS_RHR renamed TRIMS_RHR_PE4
- net TRIMS_RVD renamed TRIMS_RVD_PC3
- net TRIMS_RVU renamed TRIMS_RVU_PC2
- net USB_DM renamed USB_DM_PA11
- net USB_DP renamed USB_DP_PA12
- net USB_VBUS renamed USB_VBUS_PA9
- removed net ADC_POT1: IC1MCU.PA6
- removed net ADC_POT2: IC1MCU.PB0
- removed net ENC_A: IC1MCU.PE9
- removed net ENC_B: IC1MCU.PE11
- removed net EXTMODULE_PWR: IC1MCU.PD8
- removed net EXTMODULE_TX: IC1MCU.PA7
- removed net INTMODULE_PWR: IC1MCU.PC6
- removed net INTMODULE_TX: IC1MCU.PA10
- removed net KEYS_ENTER: IC1MCU.PE10
- removed net KEYS_EXIT: IC1MCU.PD2
- removed net KEYS_MENU: IC1MCU.PD7
- removed net KEYS_PAGE: IC1MCU.PD3
- removed net LCD_NCS: IC1MCU.PA15
- new net ADC_POT1_PA6: IC1MCU.PA6, PAD47.P
- new net ADC_POT2_PB0: IC1MCU.PB0, PAD48.P
- new net ENC_A_PE9: IC1MCU.PE9, PAD40.P
- new net ENC_B_PE11: IC1MCU.PE11, PAD41.P
- new net EXTMODULE_PWR_PD8: IC1MCU.PD8, PAD45.P
- new net EXTMODULE_TX_PA7: IC1MCU.PA7, PAD44.P
- new net INTMODULE_PWR_PC6: IC1MCU.PC6, PAD42.P
- new net INTMODULE_TX_PA10: IC1MCU.PA10, PAD43.P
- new net KEYS_ENTER_PE10: IC1MCU.PE10, PAD39.P
- new net KEYS_EXIT_PD2: IC1MCU.PD2, PAD38.P
- new net KEYS_MENU_PD7: IC1MCU.PD7, PAD36.P
- new net KEYS_PAGE_PD3: IC1MCU.PD3, PAD37.P
- new net LCD_NCS_PA15: IC1MCU.PA15, PAD22.P
- new net N$7: PAD46.P
- net SWITCHES_A_H: now also IC1MCU.PE13; no longer IC1MCU.PB5
Other:
- moved on the sheet: PAD21, PAD22, PAD23

Commit message: scheme & photo
Other:
- note added: "as general gpio (input), not vbus"
Changed lines of the file:
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@@
 <sheet>
 <plain>
+<text x="-99.06" y="-81.28" size="1.778" layer="91">as general gpio (input), not vbus</text>
 </plain>
 <instances>
