File: lcd.sch (EAGLE design)
At the start: 12 parts, among them X1 FH12-30S-0.5SH

Commit message: lcd
Parts:
- added PAD1, PAD2, PAD3, PAD4, PAD5, PAD6, PAD7: WIREPADSMD5-2,5, wirepad:WIREPADSMD5-2,5
Connections:
- removed net N$1: C10.1, C11.1, X1-1.1, X1-17.1, X1-20.1, X1-21.1, X1-22.1, X1-23.1, X1-24.1, X1-25.1, X1-26.1, X1-27.1
- removed net N$4: C10.2, C11.2, C4.2, C5.2, C6.2, C7.2, C8.2, C9.2, X1-16.1, X1-2.1, X1-3.1
- new net GND: C10.2, C11.2, C4.2, C5.2, C6.2, C7.2, C8.2, C9.2, PAD6.P, X1-16.1, X1-2.1, X1-3.1
- new net VCC: C10.1, C11.1, PAD7.P, X1-1.1, X1-17.1, X1-20.1, X1-21.1, X1-22.1, X1-23.1, X1-24.1, X1-25.1, X1-26.1, X1-27.1
- net LCD_A0_PC11: now also PAD3.P
- net LCD_CLK_PC10: now also PAD2.P
- net LCD_MOSI_PC12: now also PAD1.P
- net LCD_NCS_PA15: now also PAD5.P
- net LCD_RST_PD12: now also PAD4.P
Changed lines of the file:
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@@
 <part name="C10" library="rcl" library_urn="urn:adsk.eagle:library:334" deviceset="C-EU" device="C0805" package3d_urn="urn:adsk.eagle:package:23617/2"/>
 <part name="C11" library="rcl" library_urn="urn:adsk.eagle:library:334" deviceset="C-EU" device="C0805" package3d_urn="urn:adsk.eagle:package:23617/2"/>
+<part name="PAD1" library="wirepad" library_urn="urn:adsk.eagle:library:412" deviceset="WIREPAD" device="SMD5-2,5" package3d_urn="urn:adsk.eagle:package:30845/1"/>
+<part name="PAD2" library="wirepad" library_urn="urn:adsk.eagle:library:412" deviceset="WIREPAD" device="SMD5-2,5" package3d_urn="urn:adsk.eagle:package:30845/1"/>
+<part name="PAD3" library="wirepad" library_urn="urn:adsk.eagle:library:412" deviceset="WIREPAD" device="SMD5-2,5" package3d_urn="urn:adsk.eagle:package:30845/1"/>
+<part name="PAD4" library="wirepad" library_urn="urn:adsk.eagle:library:412" deviceset="WIREPAD" device="SMD5-2,5" package3d_urn="urn:adsk.eagle:package:30845/1"/>
+<part name="PAD5" library="wirepad" library_urn="urn:adsk.eagle:library:412" deviceset="WIREPAD" device="SMD5-2,5" package3d_urn="urn:adsk.eagle:package:30845/1"/>
+<part name="PAD6" library="wirepad" library_urn="urn:adsk.eagle:library:412" deviceset="WIREPAD" device="SMD5-2,5" package3d_urn="urn:adsk.eagle:package:30845/1"/>
+<part name="PAD7" library="wirepad" library_urn="urn:adsk.eagle:library:412" deviceset="WIREPAD" device="SMD5-2,5" package3d_urn="urn:adsk.eagle:package:30845/1"/>
 </parts>
 <sheets>
@@
 <attribute name="VALUE" x="128.016" y="-2.921" size="1.778" layer="96" rot="R180"/>
 </instance>
+<instance part="PAD1" gate="G$1" x="142.24" y="-25.4" smashed="yes" rot="R180"/>
+<instance part="PAD2" gate="G$1" x="142.24" y="-27.94" smashed="yes" rot="R180"/>
+<instance part="PAD3" gate="G$1" x="142.24" y="-30.48" smashed="yes" rot="R180"/>
+<instance part="PAD4" gate="G$1" x="142.24" y="-33.02" smashed="yes" rot="R180"/>
+<instance part="PAD5" gate="G$1" x="142.24" y="-35.56" smashed="yes" rot="R180"/>
+<instance part="PAD6" gate="G$1" x="142.24" y="0" smashed="yes" rot="R180"/>
+<instance part="PAD7" gate="G$1" x="142.24" y="-12.7" smashed="yes" rot="R180"/>
 </instances>
 <busses>
 </busses>
 <nets>
-<net name="N$1" class="0">
+<net name="VCC" class="0">
 <segment>
 <pinref part="X1" gate="-20" pin="1"/>
@@
 <pinref part="C10" gate="G$1" pin="1"/>
 <wire x1="124.46" y1="-12.7" x2="129.54" y2="-12.7" width="0.1524" layer="91"/>
-<wire x1="129.54" y1="-12.7" x2="139.7" y2="-12.7" width="0.1524" layer="91"/>
 <wire x1="124.46" y1="-10.16" x2="124.46" y2="-12.7" width="0.1524" layer="91"/>
 <junction x="124.46" y="-12.7"/>
@@
 <wire x1="129.54" y1="-10.16" x2="129.54" y2="-12.7" width="0.1524" layer="91"/>
 <junction x="129.54" y="-12.7"/>
+<pinref part="PAD7" gate="G$1" pin="P"/>
+<wire x1="129.54" y1="-12.7" x2="139.7" y2="-12.7" width="0.1524" layer="91"/>
+<label x="144.78" y="-12.7" size="1.778" layer="95"/>
 </segment>
 </net>
@@
 <wire x1="101.6" y1="-5.08" x2="101.6" y2="-25.4" width="0.1524" layer="91"/>
 <wire x1="101.6" y1="-25.4" x2="139.7" y2="-25.4" width="0.1524" layer="91"/>
-<label x="142.24" y="-25.4" size="1.778" layer="95"/>
+<label x="144.78" y="-25.4" size="1.778" layer="95"/>
+<pinref part="PAD1" gate="G$1" pin="P"/>
 </segment>
 </net>
@@
 <wire x1="99.06" y1="-7.62" x2="99.06" y2="-27.94" width="0.1524" layer="91"/>
 <wire x1="99.06" y1="-27.94" x2="139.7" y2="-27.94" width="0.1524" layer="91"/>
-<label x="142.24" y="-27.94" size="1.778" layer="95"/>
+<label x="144.78" y="-27.94" size="1.778" layer="95"/>
+<pinref part="PAD2" gate="G$1" pin="P"/>
 </segment>
 </net>
@@
 <pinref part="X1" gate="-28" pin="1"/>
 <wire x1="81.28" y1="-30.48" x2="139.7" y2="-30.48" width="0.1524" layer="91"/>
-<label x="142.24" y="-30.48" size="1.778" layer="95"/>
+<label x="144.78" y="-30.48" size="1.778" layer="95"/>
+<pinref part="PAD3" gate="G$1" pin="P"/>
 </segment>
 </net>
@@
 <pinref part="X1" gate="-29" pin="1"/>
 <wire x1="81.28" y1="-33.02" x2="139.7" y2="-33.02" width="0.1524" layer="91"/>
-<label x="142.24" y="-33.02" size="1.778" layer="95"/>
+<label x="144.78" y="-33.02" size="1.778" layer="95"/>
+<pinref part="PAD4" gate="G$1" pin="P"/>
 </segment>
 </net>
@@
 <pinref part="X1" gate="-30" pin="1"/>
 <wire x1="81.28" y1="-35.56" x2="139.7" y2="-35.56" width="0.1524" layer="91"/>
-<label x="142.24" y="-35.56" size="1.778" layer="95"/>
+<label x="144.78" y="-35.56" size="1.778" layer="95"/>
+<pinref part="PAD5" gate="G$1" pin="P"/>
 </segment>
 </net>
@@
 </segment>
 </net>
-<net name="N$4" class="0">
+<net name="GND" class="0">
 <segment>
 <pinref part="C8" gate="G$1" pin="2"/>
@@
 <junction x="86.36" y="0"/>
 <wire x1="124.46" y1="0" x2="129.54" y2="0" width="0.1524" layer="91"/>
-<wire x1="129.54" y1="0" x2="139.7" y2="0" width="0.1524" layer="91"/>
 <wire x1="129.54" y1="20.32" x2="129.54" y2="0" width="0.1524" layer="91"/>
 <junction x="129.54" y="0"/>
@@
 <pinref part="C11" gate="G$1" pin="2"/>
 <wire x1="129.54" y1="-2.54" x2="129.54" y2="0" width="0.1524" layer="91"/>
-</segment>
-</net>
+<pinref part="PAD6" gate="G$1" pin="P"/>
+<wire x1="129.54" y1="0" x2="139.7" y2="0" width="0.1524" layer="91"/>
+<label x="144.78" y="0" size="1.778" layer="95"/>
+</segment>
+</net>
